File: device_circuit_2/device_circuit_2_versionInforme.kicad_sch (KiCad schematic)
At the start: 13 parts, among them J1 DIGITAL INPUT, J2 Conn_01x15_Male, J2 GND, J3 Conn_01x15_Male, J4 Conn_01x08_Male, J5 Conn_01x08_Male, J6 MICRO STEP, J6 Screw_Terminal_01x04, J7 ENABLE MOTOR, J8 Screw_Terminal_01x02

Commit message: actualizado repo
Other:
- moved on the sheet: C3, C4, J6, J8
