File: power5-5/power5-5_version_informe.kicad_sch (KiCad schematic)
At the start: 16 parts, among them J1 AC INPUT, J2 DEVICE VCC, J3 MOTOR VCC, U1 LM7805, U2 LM7905

Commit message: actualizado repo
Connections:
- net GND: no longer C5.2, C6.1, D3.1 (K), J2.2 (Pin_2), R1.1, U1.2 (GND), U2.1 (GND)
- net at C1.1, C3.1, J3.3 (Pin_3)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: now also D1.1 (+)
- new net: C5.2, C6.1, D3.1 (K), J2.2 (Pin_2), R1.1, U1.2 (GND), U2.1 (GND)
Other:
- moved on the sheet: C1, C2, C3, C4, D1, J1
